Commit message: calude off pi cleanup og debug

File: src/wg_utilities/nav2/static_tf.urdf (robot description, URDF)
Before this commit: robot tracked_robot_minimal, 3 links, 2 joints
Links:
- added link servo_link; visual box size=0.04 0.04 0.04
Joints:
- added joint base_to_servo: type fixed, parent base_link, child servo_link, origin xyz=0.12 0.0 0.08 rpy=0 0 0
